File: _autosave-io.kicad_sch (KiCad schematic)
At the start: 56 parts, among them J3 Micro_SD_Card, J4 LASER, J6 TT143AMC12C, Q1 BSS214NW, U1 LSM6DSOXTR, U10 MAX30102, U11 TPS65631W, U12 TXB0102YZP, U14 LIS3MDL, U16 DRV2605LDGS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

Commit message: done with stm, going back to esp
Parts:
- added R9: 0, symbol Device:R
Connections:
- net GND: now also R9.1; no longer J6.24 (MTP_PWR)
- net SCL1 renamed IMU_SCL
- removed net SCL2: U10.2 (SCL), U14.1 (SCL/SPC), U16.2 (SCL), U7.2 (SCL)
- net SCL3 renamed TP_SCL
- net SDA1 renamed IMU_SDA
- removed net SDA2: U10.3 (SDA), U14.11 (SDA/SDI/SDO), U16.3 (SDA), U7.4 (SDA)
- net SDA3 renamed TP_SDA
- new net: J6.24 (MTP_PWR), R9.2
- new net ALT_SCL: U7.2 (SCL)
- new net ALT_SDA: U7.4 (SDA)
- new net HBT_SCL: U10.2 (SCL)
- new net HBT_SDA: U10.3 (SDA)
- new net MAG_SCL: U14.1 (SCL/SPC)
- new net MAG_SDA: U14.11 (SDA/SDI/SDO)
- new net MTR_SCL: U16.2 (SCL)
- new net MTR_SDA: U16.3 (SDA)
Other:
- moved on the sheet: C19, C20, C26, C27, C28, C32, C33, C35, C36, C38, C39, C40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
