File: stm_mcu.kicad_sch (KiCad schematic)
At the start: 63 parts, among them J3 Micro_SD_Card, J8 SWD, U15 TXS02612RTW, U3 STM32H7S7L8H6H, U5 APS256XXN-OBR-BG, Y3 32.768kHz, Y4 40MHz(10ppm)

Commit message: done with stm, going back to esp
Parts:
- removed C19: 10uF, symbol Device:C_Small
- removed C20: 100nF, symbol Device:C_Small
- removed J3: Micro_SD_Card, Connector_Card:microSD_HC_Molex_104031-0811, symbol Connector:Micro_SD_Card
Connections:
- net SD_DEV_CLK renamed SD_CLK
- net SD_DEV_CMD renamed SD_CMD
- net SD_DEV_D0 renamed SD_D0
- net SD_DEV_D1 renamed SD_D1
- net SD_DEV_D2 renamed SD_D2
- net SD_DEV_D3 renamed SD_D3
