File: _autosave-watch-pcb.kicad_pcb (KiCad board)
At the start: 6 copper layers, 42 x 42 mm, 171 parts, among them J1 NFP-ELV0832B, J2 USB_C_Receptacle, J3 ESP_ANT, J4 LASER, J5 Micro_SD_Card, J6 TT143AMC12C, Q1 BSS214NW, SW1 B3U-3000P, SW3 SW_Push, SW4 SW_Push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

Commit message: layout done probably
Parts:
- moved C42 0.90 mm to (151.3, 76.0), turned to 180 degrees
- moved R36 0.81 mm to (152.8, 103.2)
- moved C41 0.65 mm to (148.7, 72.5), turned to -90 degrees
- moved J1 0.14 mm to (155.0, 92.1)
- moved C79 0.05 mm to (144.8, 93.2)
- moved U13 0.05 mm to (149.1, 93.7)
Routing:
- net /ESP MCU/EXT_IO6: track 3.45 -> 0.04 mm
- net /ESP MCU/RTC_P: track 0.00 -> 2.28 mm
- net /ESP MCU/RTC_N: track 0.00 -> 2.28 mm
- net /ESP MCU/MEM_CLK: track 11.8 -> 13.5 mm
- net /ESP MCU/MEM_D3: track 13.6 -> 12.6 mm, vias 1 -> 2
- net /ESP MCU/MEM_D0: vias 1 -> 2
