File: esp_mcu.kicad_sch (KiCad schematic)
At the start: 55 parts, among them J5 ESP_ANT, U18 TCA9535MRGER, U3 MX25UM51245GXDI00, U5 S80KS5123GABHV020, U9 ESP32-S3, Y1 32.768kHz, Y2 40MHz(10ppm)

Commit message: no more daughter probably
Parts:
- R21: renamed from R39; footprint PCM_Resistor_SMD_AKL:R_0402_1005Metric -> Capacitor_SMD:C_0402_1005Metric
- renumbered C25 to C21, C34 to C22, C79 to C23, C78 to C24, C37 to C25, C41 to C26, C81 to C27, C82 to C28, C83 to C29, C84 to C30, C30 to C31, C31 to C32, C46 to C33, C43 to C34, C47 to C35, C44 to C36, C48 to C37, C60 to C38, C61 to C39, C77 to C40, C29 to C41, C45 to C43, C86 to C44, C87 to C45, C75 to C46, C76 to C47, J5 to J3, L5 to L4, L6 to L5, L9 to L6, R46 to R19, R40 to R20, R31 to R22, R32 to R23, R53 to R24, R33 to R25, R34 to R26, R41 to R27, R35 to R28, R42 to R29, R43 to R30, R44 to R31, R36 to R32, R45 to R33, R37 to R34, R38 to R35, U3 to U5, U5 to U6, U9 to U7, U18 to U8

Commit message: basically done with board layout, gonna try to do a smaller one (47->42mm diameter)
Parts:
- removed JP1: RESET=LOW, Jumper:SolderJumper-2_P1.3mm_Open_RoundedPad1.0x1.5mm, symbol Jumper:SolderJumper_2_Open
- removed R22: 10k, Resistor_SMD:R_0402_1005Metric, symbol Device:R
- removed R34, R35: 0, Resistor_SMD:R_0402_1005Metric, symbol Device:R
- added R5, R6: 0, Resistor_SMD:R_0402_1005Metric, symbol Device:R
- added R50, R51: 10k, Resistor_SMD:R_0402_1005Metric, symbol Device:R
- added TP1: BOOT, TestPoint:TestPoint_Pad_D2.0mm, symbol Connector:TestPoint
- added TP2: RST, TestPoint:TestPoint_Pad_D2.0mm, symbol Connector:TestPoint
- added TP3: GND, TestPoint:TestPoint_Pad_D2.0mm, symbol Connector:TestPoint
- added TP4: RX, TestPoint:TestPoint_Pad_D2.0mm, symbol Connector:TestPoint
- added TP5: TX, TestPoint:TestPoint_Pad_D2.0mm, symbol Connector:TestPoint
- C21, C22: footprint Capacitor_SMD:C_0201_0603Metric -> Capacitor_SMD:C_0402_1005Metric
- L4: footprint Inductor_SMD:L_0201_0603Metric -> Inductor_SMD:L_0402_1005Metric
- L5: footprint Inductor_SMD:L_0805_2012Metric -> Inductor_SMD:L_0402_1005Metric
- L6: footprint Inductor_SMD:L_Coilcraft_XFL2010 -> Capacitor_SMD:C_0402_1005Metric
Connections:
- net BOOTSEL is gone; now on net I2S_SCK: U7.52 (GPIO46)
- net RX is gone; now on net IO9: U7.50 (U0RXD)
- net TX is gone; now on net IO8: R25.1
- net +1V8: now also C24.2; no longer C24.1
- net +3V3: now also C42.2, C43.2, U7.20 (VDD3P3_RTC), U7.46 (VDD3P3_CPU), R51.1
- net EN: now also TP2.1
- net GND: now also C24.1, R50.1, TP3.1; no longer C24.2
- net I2C0_SCL: now also TP1.1
- net I2S_SCK: now also R50.2; no longer U7.51 (GPIO45)
- net IO8: now also TP5.1; no longer U7.25 (GPIO19)
- net IO9: now also TP4.1; no longer U7.26 (GPIO20)
- net MEM_CLK: now also R31.1; no longer R32.1
- net MEM_D0: now also R33.1
- net MEM_D1: now also R32.1
- net MEM_D2: now also R30.1; no longer R28.1
- net MEM_D3: now also R29.1; no longer R26.1
- net MEM_D4: now also R5.2; no longer R27.1
- net MEM_D5: now also R6.2; no longer R29.1
- net MEM_D6: now also R26.2; no longer R30.1
- net MEM_D7: now also R27.2; no longer R31.1
- net MEM_DQS: now also R28.2; no longer R33.1
- net SD_CMD: now also U7.45 (MTDO); no longer U7.37 (SPICLK_P)
- net SD_D0: now also U7.47 (MTDI); no longer U7.44 (MTCK)
- net SD_D1: now also U7.48 (MTMS); no longer U7.45 (MTDO)
- net SD_D2: now also U7.37 (SPICLK_P); no longer U7.47 (MTDI)
- net SD_D3: now also U7.44 (MTCK); no longer U7.48 (MTMS)
- net at U7.35 (SPID): now also R33.2
- net at R29.2: now also U7.30 (SPIHD); no longer U7.39 (GPIO34)
- net at U7.34 (SPIQ): now also R32.2
- net at U7.40 (GPIO35): now also R26.1; no longer R30.2
- net at U7.38 (GPIO33): now also R5.1; no longer R27.2
- net at R31.2: now also U7.33 (SPICLK); no longer U7.41 (GPIO36)
- net at U7.42 (GPIO37): now also R28.1; no longer R33.2
- net at U7.31 (SPIWP): now also R30.2; no longer R28.2
- new net: R6.1, U7.39 (GPIO34)
- new net: R27.1, U7.41 (GPIO36)
- new net I2S_WS: R51.2, U7.51 (GPIO45)
- new net USB_DM: U7.25 (GPIO19)
- new net USB_DP: U7.26 (GPIO20)
Other:
- note added: "LQG15HN2N0C02D"
- note added: "LRC0402CS2N7GV001T"
- note removed: "LQP03TN2N7B02D"
- moved on the sheet: C24

Commit message: layout done probably
Parts:
- removed R26, R27, R28, R29, R30, R31, R32, R33, R5, R6: 0, Resistor_SMD:R_0402_1005Metric, symbol Device:R
- removed R51: 10k, Resistor_SMD:R_0402_1005Metric, symbol Device:R
Connections:
- net IO9 is gone; now on net IO8: TP4.1, U7.50 (U0RXD)
- net +3V3: now also U7.51 (GPIO45)
- net I2S_SD: now also U7.24 (GPIO18); no longer U7.43 (GPIO38)
- net I2S_WS: now also U7.43 (GPIO38); no longer U7.51 (GPIO45)
- net IO7: now also R25.1, TP5.1; no longer U7.24 (GPIO18)
- net IO8: no longer R25.1, TP5.1
- net MEM_CLK: now also U7.33 (SPICLK)
- net MEM_D0: now also U7.35 (SPID)
- net MEM_D1: now also U7.34 (SPIQ)
- net MEM_D2: now also U7.31 (SPIWP)
- net MEM_D3: now also U7.30 (SPIHD)
- net MEM_D4: now also U7.38 (GPIO33)
- net MEM_D5: now also U7.39 (GPIO34)
- net MEM_D6: now also U7.40 (GPIO35)
- net MEM_D7: now also U7.41 (GPIO36)
- net MEM_DQS: now also U7.42 (GPIO37)

Commit message: finally routed the memory :D
Parts:
- removed C35, C37, C38, C42, C43: 100nF, Capacitor_SMD:C_0402_1005Metric, symbol Device:C_Small
- removed C36, C39: 1uF, Capacitor_SMD:C_0402_1005Metric, symbol Device:C_Small
- removed C40: 10uF, Capacitor_SMD:C_0402_1005Metric, symbol Device:C_Small
- removed R21: R, Capacitor_SMD:C_0402_1005Metric, symbol Device:R
- removed R25: 499, Resistor_SMD:R_0402_1005Metric, symbol Device:R
- removed TP1: BOOT, TestPoint:TestPoint_Pad_D2.0mm, symbol Connector:TestPoint
- removed TP2: RST, TestPoint:TestPoint_Pad_D2.0mm, symbol Connector:TestPoint
- removed TP3: GND, TestPoint:TestPoint_Pad_D2.0mm, symbol Connector:TestPoint
- removed TP4: RX, TestPoint:TestPoint_Pad_D2.0mm, symbol Connector:TestPoint
- removed TP5: TX, TestPoint:TestPoint_Pad_D2.0mm, symbol Connector:TestPoint
- removed U7: ESP32-S3, Package_DFN_QFN:QFN-56-1EP_7x7mm_P0.4mm_EP4x4mm_ThermalVias, symbol MCU_Espressif:ESP32-S3
- added C10, C11, C13, C14, C16: 100nF, Capacitor_SMD:C_0402_1005Metric, symbol Device:C_Small
- added C17, C4, C9: 1uF, Capacitor_SMD:C_0402_1005Metric, symbol Device:C_Small
- added Q2, Q3: BSS138, Package_TO_SOT_SMD:SOT-23, symbol Transistor_FET:BSS138
- added R1: 10k, Resistor_SMD:R_0402_1005Metric, symbol Device:R
- added R35, R37, R44, R51, R52, R53, R54, R55, R8: 0, Resistor_SMD:R_0201_0603Metric, symbol Device:R
- added SW8: BOOT, Button_Switch_SMD:SW_SPST_CK_KXT3, symbol Switch:SW_Push
- added U11: ESP32-S3, Package_DFN_QFN:QFN-56-1EP_7x7mm_P0.4mm_EP4x4mm_ThermalVias, symbol MCU_Espressif:ESP32-S3
- C34: value 1uF -> 10uF
- L5: value 2nH -> LQG15HN2N0C02D
- R19, R20: value 10k -> 100k
- R50: value 10k -> 0; footprint Resistor_SMD:R_0402_1005Metric -> Resistor_SMD:R_0201_0603Metric
Connections:
- net +1V8: now also C10.1, C9.1, U11.29 (VDD_SPI)
- net +3V3: now also C33.1, C34.1, C11.1, C13.1, C16.1, C17.1, C4.1, SW8.1, U11.20 (VDD3P3_RTC), U11.46 (VDD3P3_CPU), U11.55 (VDDA), U11.56 (VDDA); no longer C33.2, C34.2
- net CLK_N: now also U11.53 (XTAL_N)
- net CLK_P: now also U11.54 (XTAL_P)
- net ESP_ANT: now also U11.1 (LNA_IN)
- net EXT_INT: now also U11.27 (GPIO21)
- net FSPI_CLK: now also U11.17 (GPIO12)
- net FSPI_CS: now also U11.15 (GPIO10)
- net FSPI_D: now also U11.16 (GPIO11)
- net FSPI_HD: now also U11.14 (GPIO9)
- net FSPI_Q: now also U11.18 (GPIO13)
- net FSPI_WP: now also U11.19 (GPIO14)
- net GND: now also C33.2, C34.2, C10.2, C11.2, C13.2, C14.2, C16.2, C17.2, C4.2, C9.2, Q2.2 (S), Q3.2 (S), R1.1, U11.57 (GND); no longer C33.1, C34.1, R50.1
- net I2C0_SCL: now also U8.19 (SCL); no longer U8.20 (SDA)
- net I2C0_SDA: now also U8.20 (SDA); no longer U8.19 (SCL)
- net I2S_SCK: now also U11.45 (MTDO); no longer R50.2
- net I2S_SD: now also U11.43 (GPIO38)
- net I2S_WS: now also U11.44 (MTCK)
- net IO1: now also U11.9 (GPIO4)
- net IO2: now also U11.10 (GPIO5)
- net IO3: now also U11.11 (GPIO6)
- net IO4: now also U11.12 (GPIO7)
- net IO5: now also U11.13 (GPIO8)
- net IO6: now also U11.23 (GPIO17)
- net IO7: now also U11.24 (GPIO18)
- net IO8: now also U11.37 (SPICLK_P)
- net MEM_CLK: now also R52.2
- net MEM_CS0: now also U11.32 (SPICS0)
- net MEM_CS1: now also U11.28 (SPICS1)
- net MEM_D0: now also R54.2
- net MEM_D1: now also R53.2
- net MEM_D2: now also R51.2
- net MEM_D3: now also R50.2
- net MEM_D4: now also R8.2
- net MEM_D5: now also R35.2
- net MEM_D6: now also R37.2
- net MEM_D7: now also R44.2
- net MEM_DQS: now also R55.2
- net RTC_N: now also U11.22 (XTAL_32K_N)
- net RTC_P: now also U11.21 (XTAL_32K_P)
- net SD_CLK: now also U11.50 (U0RXD)
- net SD_CMD: now also U11.49 (U0TXD)
- net SD_D0: now also U11.51 (GPIO45)
- net SD_D1: now also Q2.3 (D), U11.52 (GPIO46)
- net SD_D2: now also U11.47 (MTDI)
- net SD_D3: now also U11.48 (MTMS)
- net at C41.1, R23.2: now also U11.4 (CHIP_PU)
- net at L5.1: now also C14.1, U11.2 (VDD3P3), U11.3 (VDD3P3)
- new net: R50.1, U11.30 (SPIHD)
- new net: R51.1, U11.31 (SPIWP)
- new net: R52.1, U11.33 (SPICLK)
- new net: R53.1, U11.34 (SPIQ)
- new net: R54.1, U11.35 (SPID)
- new net: R8.1, U11.38 (GPIO33)
- new net: R35.1, U11.39 (GPIO34)
- new net: R37.1, U11.40 (GPIO35)
- new net: R44.1, U11.41 (GPIO36)
- new net: R55.1, U11.42 (GPIO37)
- new net BOOT: Q2.1 (G), Q3.1 (G), R1.2, SW8.2
- new net IO9: U11.36 (SPICLK_N)
- new net MCU_SCL: Q3.3 (D), U11.5 (GPIO0)
- new net MCU_SDA: U11.6 (GPIO1)
- new net RTC_SCL: U11.7 (GPIO2)
- new net RTC_SDA: U11.8 (GPIO3)
- new net USB_D+: U11.26 (GPIO20/USB_D+)
- new net USB_D-: U11.25 (GPIO19/USB_D-)
Other:
- note added: "500 mA max"
- note added: "512Mb/64MB 200MHz DDR OPI PSRAM 30mA typ 40mA max"
- note added: "gp43 gp44"
- note removed: "512Mb/64MB 200MHz DDR OPI PSRAM"
- note removed: "LQG15HN2N0C02D"
- note removed: "gp44 gp43"
- moved on the sheet: C21, C22, C31, C32, C33, C41, J3, L4, L5, R23, Y1
