File: usb_power.kicad_sch (KiCad schematic)
At the start: 45 parts, among them J2 USB_C_Receptacle, U17 TPS62161DSG, U2 TPS63021, U4 BQ27427YZFR, U6 BQ25628E

Commit message: quicksaving pcb bc im gonna redo it
Parts:
- added C18, C21, C22: 22uF, Capacitor_SMD:C_0603_1608Metric, symbol Device:C_Small
Connections:
- net +BATT: now also C18.1, C21.1, C22.1
- net GND: now also C18.2, C21.2, C22.2
Other:
- moved on the sheet: BT1, C11, C14, C15, C16, C17, C88, C89, C90, D5, D6, D7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

Commit message: no more daughter probably
Parts:
- added C79, C80: 10uF, Capacitor_SMD:C_0805_2012Metric, symbol Device:C_Small
- C12: renamed from C88; footprint Capacitor_SMD:C_0402_1005Metric -> Capacitor_SMD:C_0603_1608Metric
- C15: renamed from C90; footprint Capacitor_SMD:C_0402_1005Metric -> Capacitor_SMD:C_0805_2012Metric
- C16: renamed from C49; footprint Capacitor_SMD:C_0402_1005Metric -> Capacitor_SMD:C_0603_1608Metric
- C17: renamed from C59; footprint Capacitor_SMD:C_0402_1005Metric -> Capacitor_SMD:C_0603_1608Metric
- C2: renamed from C4; footprint Capacitor_SMD:C_0603_1608Metric -> Capacitor_SMD:C_0402_1005Metric
- C3: renamed from C89; footprint Capacitor_SMD:C_0402_1005Metric -> Capacitor_SMD:C_0603_1608Metric
- L2: renamed from L4; footprint (none) -> Inductor_SMD:L_1008_2520Metric
- R15: renamed from R25; footprint (none) -> Resistor_SMD:R_0603_1608Metric
- U4: footprint Package_BGA:Texas_DSBGA-9_1.62mmx1.58mm_Layout3x3_P0.5mm -> Package_BGA:Texas_DSBGA-9_1.62x1.58mm_Layout3x3_P0.5mm
- renumbered C14 to C1, C21 to C10, C22 to C11, C1 to C13, C2 to C14, C5 to C18, C11 to C19, C15 to C20, C17 to C4, C16 to C5, C7 to C6, C8 to C7, C10 to C8, C18 to C9, D5 to D3, D6 to D4, D7 to D5, D3 to D6, D2 to D7, D4 to D8, R15 to R10, R61 to R11, R60 to R12, R56 to R13, R57 to R14, R11 to R16, R12 to R17, R19 to R18, R13 to R7, R14 to R8, R62 to R9, TH2 to TH1, U2 to U1, U6 to U2, U17 to U3
Connections:
- net +VSW: now also C79.1, C80.1
- net GND: now also C79.2, C80.2
Other:
- note added: "CIGT252010EH1R0MNE"
- moved on the sheet: R16, R17, R9

Commit message: basically done with board layout, gonna try to do a smaller one (47->42mm diameter)
Parts:
- added SW1: B3U-3000P, Button_Switch_SMD:SW_SPST_B3U-3000P, symbol Switch:SW_Push
- L1: value 1.5uH -> XFL4020-152ME; footprint custom-lib:XFL4020-152ME -> Inductor_SMD:L_Coilcraft_XxL4040
Connections:
- net +BATT: now also C15.2; no longer C15.1
- net GND: now also C15.1, SW1.2; no longer C15.2
- net ILIM: no longer names the net of R9.1, U2.4 (ILIM)
- net POWER_BTN: no longer names the net of U2.7 (QON)
- net POWER_BTN: now also SW1.1
Other:
- note removed: "500 mA (2500/R)"
- note removed: "XFL4020-152ME"
- moved on the sheet: C15, C16, C17, L3, R11, R12, R15, R9, TH1, U3

Commit message: layout done probably
Parts:
- removed D5: POWER GOOD, LED_SMD:LED_0402_1005Metric, symbol Device:LED
- removed R14: R, Resistor_SMD:R_0402_1005Metric, symbol Device:R
Connections:
- no-connect marks 11 -> 12
Changed lines of the file:
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@@
 	)
 	(junction
-		(at 251.46 50.8)
-		(diameter 0)
-		(color 0 0 0 0)
-	)
-	(junction
 		(at 39.37 40.64)
 		(diameter 0)
@@
 	)
 	(no_connect
+		(at 229.87 52.07)
+	)
+	(no_connect
 		(at 46.99 180.34)
 	)
@@
 	(wire
 		(pts
-			(xy 251.46 49.53) (xy 251.46 50.8)
-		)
-		(stroke
-			(width 0)
-			(type default)
-		)
-	)
-	(wire
-		(pts
 			(xy 46.99 142.24) (xy 46.99 143.51)
 		)
@@
 	(wire
 		(pts
-			(xy 251.46 50.8) (xy 255.27 50.8)
+			(xy 251.46 49.53) (xy 255.27 49.53)
 		)
 		(stroke
@@
 	(wire
 		(pts
-			(xy 251.46 50.8) (xy 251.46 52.07)
-		)
-		(stroke
-			(width 0)
-			(type default)
-		)
-	)
-	(wire
-		(pts
-			(xy 229.87 52.07) (xy 236.22 52.07)
-		)
-		(stroke
-			(width 0)
-			(type default)
-		)
-	)
-	(wire
-		(pts
 			(xy 201.93 52.07) (xy 201.93 49.53)
 		)
@@
 	(symbol
 		(lib_id "power:+3V3")
-		(at 255.27 50.8 270)
+		(at 255.27 49.53 270)
 		(unit 1)
 		(exclude_from_sim no)
@@
 		(fields_autoplaced yes)
 		(property "Reference" "#PWR021"
-			(at 251.46 50.8 0)
+			(at 251.46 49.53 0)
 			(effects
 				(font
@@
 		)
 		(property "Value" "+3V3"
-			(at 259.08 50.7999 90)
+			(at 259.08 49.5299 90)
 			(effects
 				(font
@@
 		)
 		(property "Footprint" ""
-			(at 255.27 50.8 0)
+			(at 255.27 49.53 0)
 			(effects
 				(font
@@
 		)
 		(property "Datasheet" ""
-			(at 255.27 50.8 0)
+			(at 255.27 49.53 0)
 			(effects
 				(font
@@
 		)
 		(property "Description" ""
-			(at 255.27 50.8 0)
+			(at 255.27 49.53 0)
 			(effects
 				(font
@@
 	)
 	(symbol
-		(lib_id "Device:LED")
-		(at 240.03 52.07 0)
-		(unit 1)
-		(exclude_from_sim no)
-		(in_bom yes)
-		(on_board yes)
-		(dnp no)
-		(property "Reference" "D5"
-			(at 243.84 53.34 0)
-			(effects
-				(font
-					(size 1.27 1.27)
-				)
-			)
-		)
-		(property "Value" "POWER GOOD"
-			(at 243.84 55.88 0)
-			(effects
-				(font
-					(size 1.27 1.27)
-				)
-			)
-		)
-		(property "Footprint" "LED_SMD:LED_0402_1005Metric"
-			(at 240.03 52.07 0)
-			(effects
-				(font
-					(size 1.27 1.27)
-				)
-				(hide yes)
-			)
-		)
-		(property "Datasheet" "~"
-			(at 240.03 52.07 0)
-			(effects
-				(font
-					(size 1.27 1.27)
-				)
-				(hide yes)
-			)
-		)
-		(property "Description" ""
-			(at 240.03 52.07 0)
-			(effects
-				(font
-					(size 1.27 1.27)
-				)
-				(hide yes)
-			)
-		)
-		(pin "1"
-		)
-		(pin "2"
-		)
-		(instances
-			(project "watch-pcb"
-				(path "/b7b86b03-b0df-4b4e-be1d-606605306dad/ac5844b2-70bd-47c8-b13a-e6d4bebf0e4d"
-					(reference "D5")
-					(unit 1)
-				)
-			)
-		)
-	)
-	(symbol
 		(lib_id "Device:C_Small")
 		(at 207.01 24.13 270)
@@
 		(dnp no)
 		(property "Reference" "R13"
-			(at 254 49.53 90)
+			(at 252.222 48.26 90)
 			(effects
 				(font
@@
 					(unit 1)
 				)
-			)
-		)
-	)
-	(symbol
-		(lib_id "Device:R")
-		(at 247.65 52.07 90)
-		(unit 1)
-		(exclude_from_sim no)
-		(in_bom yes)
-		(on_board yes)
-		(dnp no)
-		(property "Reference" "R14"
-			(at 254 52.07 90)
-			(effects
-				(font
-					(size 1.27 1.27)
-				)
-			)
-		)
-		(property "Value" "R"
-			(at 247.65 52.07 90)
-			(effects
-				(font
-					(size 1.27 1.27)
-				)
-			)
-		)
-		(property "Footprint" "Resistor_SMD:R_0402_1005Metric"
-			(at 247.65 53.848 90)
-			(effects
-				(font
-					(size 1.27 1.27)
-				)
-				(hide yes)
-			)
-		)
-		(property "Datasheet" "~"
-			(at 247.65 52.07 0)
-			(effects
-				(font
-					(size 1.27 1.27)
-				)
-				(hide yes)
-			)
-		)
-		(property "Description" ""
-			(at 247.65 52.07 0)
-			(effects
-				(font
-					(size 1.27 1.27)
-				)
-				(hide yes)
-			)
-		)
-		(pin "1"
-		)
-		(pin "2"
-		)
-		(instances
-			(project "watch-pcb"
-				(path "/b7b86b03-b0df-4b4e-be1d-606605306dad/ac5844b2-70bd-47c8-b13a-e6d4bebf0e4d"
-					(reference "R14")
-					(unit 1)
-				)

Commit message: finally routed the memory :D
Parts:
- removed BT1: Battery, custom-lib:Battery_Connector, symbol Device:Battery
- removed C10, C11, C17, C9: 22uF, Capacitor_SMD:C_0603_1608Metric, symbol Device:C_Small
- removed C13, C14, C16: 10uF, Capacitor_SMD:C_0603_1608Metric, symbol Device:C_Small
- removed C4: 100nF, Capacitor_SMD:C_0402_1005Metric, symbol Device:C_Small
- removed R7: 180k, Resistor_SMD:R_0402_1005Metric, symbol Device:R
- removed R8: 1M, Resistor_SMD:R_0402_1005Metric, symbol Device:R
- removed U3: TPS62161DSG, Package_SON:WSON-8-1EP_2x2mm_P0.5mm_EP0.9x1.6mm_ThermalVias, symbol Regulator_Switching:TPS62161DSG
- added C35: 100nF, Capacitor_SMD:C_0402_1005Metric, symbol Device:C_Small
- added C63: 22uF, Capacitor_SMD:C_0805_2012Metric, symbol Device:C_Small
- added C64, C65: 10uF, Capacitor_SMD:C_0805_2012Metric, symbol Device:C_Small
- added C81: 4.7uF, Capacitor_SMD:C_0603_1608Metric, symbol Device:C_Small
- added C84: 10uF, Capacitor_SMD:C_0603_1608Metric, symbol Device:C_Small
- added J7: BATT+, TestPoint:TestPoint_THTPad_2.0x2.0mm_Drill1.0mm, symbol Connector:Conn_01x01_Socket
- added J8: BATT-, TestPoint:TestPoint_THTPad_2.0x2.0mm_Drill1.0mm, symbol Connector:Conn_01x01_Socket
- added R14: 100k, Resistor_SMD:R_0402_1005Metric, symbol Device:R
- added R22: 5.1k, Resistor_SMD:R_0603_1608Metric, symbol Device:R
- added R26: 0, Resistor_SMD:R_0402_1005Metric, symbol Device:R
- added R28: 200k, Resistor_SMD:R_0603_1608Metric, symbol Device:R
- added R29: 100k, Resistor_SMD:R_0603_1608Metric, symbol Device:R
- added R30: 499k, Resistor_SMD:R_0402_1005Metric, symbol Device:R
- added U17: TLV62569DDC, Package_TO_SOT_SMD:SOT-23-6, symbol Regulator_Switching:TLV62569DDC
- L2: value 1uH -> CIGT252010EH1R0MNE
- L3: value 2.2uH -> XFL4020-222ME; footprint Inductor_SMD:L_1206_3216Metric -> Inductor_SMD:L_Coilcraft_XxL4040
- R15: footprint Resistor_SMD:R_0603_1608Metric -> Resistor_SMD:R_0402_1005Metric
- R16: footprint Resistor_SMD:R_0402_1005Metric -> Resistor_SMD:R_0603_1608Metric
- R17: value 5.1k -> 100k
- SW1: value B3U-3000P -> B3U-3000P-B; footprint Button_Switch_SMD:SW_SPST_B3U-3000P -> Button_Switch_SMD:SW_SPST_B3U-3000P-B
Connections:
- net +1V8: now also C84.2, R28.1; no longer R15.1
- net +3V3: now also R15.2, R17.2, U1.3 (FB)
- net +BATT: now also C63.1, J7.1 (Pin_1)
- net +VSW: now also C64.1, C65.1, C81.1, R30.2, U17.1 (EN), U17.4 (VIN)
- net 3V3_POWER_SAVE: now also R14.1
- net BAT_LOW: now also R17.1
- net CHARGE_INT: now also R15.1
- net GND: now also J2.S1 (SHIELD), C35.2, C63.2, C64.2, C65.2, C81.2, C84.1, J8.1 (Pin_1), R14.2, R22.2, R29.2, U17.2 (GND); no longer R17.2
- net at SW1.1, U2.7 (QON): now also R26.1
- net at C3.2, U2.17 (PMID): now also C35.1
- net at L3.1: now also U17.3 (SW)
- net at J2.B5 (CC2): now also R22.1; no longer R17.1
- net 1V8_GOOD renamed 1V8G
- net 1V8G: now also R30.1, U17.5 (PG); no longer R15.2
- net USB_DM renamed USB_D-
- net USB_DP renamed USB_D+
- new net: R28.2, R29.1, U17.6 (FB)
- new net QON: R26.2
- no-connect marks 12 -> 11
Other:
- note added: "Good"
- note added: "fuse?"
- note added: "make sure vina is connected"
- note added: "pull pg to what? check.."
- note removed: "0603, 1% 1/16 W"
- note removed: "25 V Ceramic 0805"
- note removed: "6.3 V Ceramic 0805"
- note removed: "CIGT252010EH1R0MNE"
- note removed: "VLF3012ST-2R2M1R4, TDK from datasheet"
- moved on the sheet: C1, C12, C15, C19, C2, C20, C3, C5, C79, C80, D3, D4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
