File: watch-pcb.kicad_pcb (KiCad board)
At the start: 6 copper layers, 42 x 42 mm, 171 parts, among them J1 NFP-ELV0832B, J2 USB_C_Receptacle, J3 ESP_ANT, J4 LASER, J5 Micro_SD_Card, J6 TT143AMC12C, Q1 BSS214NW, SW1 B3U-3000P, SW3 SW_Push, SW4 SW_Push, SW5 SW_Push, U1 TPS63021, U10 LIS3MDL, U11 LPS22DF, U12 LSM6DSOXTR, U13 DRV2605LDGS, U14 MAX30102, U15 APDS-9306-065, U16 AP3019AK, U2 BQ25628E, U3 TPS62161DSG, U4 BQ27427YZFR, U5 MX25UM51245GXDI00, U6 S80KS5123GABHV020, U7 ESP32-S3, U8 TCA9535MRGER, U9 TPS65631W, Y1 32.768kHz, Y2 40MHz(10ppm)

Commit message: finally routed the memory :D
Parts:
- removed BT1: Battery, custom-lib:Battery_Connector
- removed C36, C39: 1uF, Capacitor_SMD:C_0402_1005Metric
- removed C37, C38, C42, C43, C53, C83: 100nF, Capacitor_SMD:C_0402_1005Metric
- removed C40: 10uF, Capacitor_SMD:C_0402_1005Metric
- removed C49: 4.7uF, Capacitor_SMD:C_0603_1608Metric
- removed J1: NFP-ELV0832B, custom-lib:Battery_Connector
- removed J4: LASER, custom-lib:LASER_connector
- removed R21: R, Capacitor_SMD:C_0402_1005Metric
- removed R25: 499, Resistor_SMD:R_0402_1005Metric
- removed R34: 10k, Resistor_SMD:R_0402_1005Metric
- removed R7: 180k, Resistor_SMD:R_0402_1005Metric
- removed SW5: SW_Push, Button_Switch_SMD:SW_SPST_B3U-3000P
- removed TP1: BOOT, TestPoint:TestPoint_Pad_D2.0mm
- removed TP2: RST, TestPoint:TestPoint_Pad_D2.0mm
- removed TP3: GND, TestPoint:TestPoint_Pad_D2.0mm
- removed TP4: RX, TestPoint:TestPoint_Pad_D2.0mm
- removed TP5: TX, TestPoint:TestPoint_Pad_D2.0mm
- removed U7: ESP32-S3, Package_DFN_QFN:QFN-56-1EP_7x7mm_P0.4mm_EP4x4mm_ThermalVias
- added C54: 100nF, Capacitor_SMD:C_0402_1005Metric, B.Cu at (152.5, 64.8)
- added C62: 100nF, Capacitor_SMD:C_0402_1005Metric, B.Cu at (152.5, 66.6)
- added C63: 22uF, Capacitor_SMD:C_0805_2012Metric, B.Cu at (147.6, 97.7)
- added C64: 10uF, Capacitor_SMD:C_0805_2012Metric, F.Cu at (156.8, 85.7)
- added C65: 10uF, Capacitor_SMD:C_0805_2012Metric, F.Cu at (154.8, 85.7)
- added C81: 4.7uF, Capacitor_SMD:C_0603_1608Metric, F.Cu at (159.7, 78.5)
- added C84: 10uF, Capacitor_SMD:C_0603_1608Metric, F.Cu at (162.8, 73.2)
- added J10: LASER-, TestPoint:TestPoint_Keystone_5015_Micro_Mini, F.Cu at (156.3, 102.0)
- added J11: MTR+, TestPoint:TestPoint_THTPad_1.5x1.5mm_Drill0.7mm, B.Cu at (152.1, 103.2)
- added J13: MTR-, TestPoint:TestPoint_THTPad_1.5x1.5mm_Drill0.7mm, B.Cu at (152.1, 100.7)
- added J7: BATT+, TestPoint:TestPoint_THTPad_2.0x2.0mm_Drill1.0mm, F.Cu at (144.9, 98.0)
- added J8: BATT-, TestPoint:TestPoint_THTPad_2.0x2.0mm_Drill1.0mm, F.Cu at (150.6, 98.0)
- added J9: LASER+, TestPoint:TestPoint_Keystone_5015_Micro_Mini, B.Cu at (156.3, 100.5)
- added Q2: BSS138, Package_TO_SOT_SMD:SOT-23, B.Cu at (132.2, 64.9)
- added Q3: BSS138, Package_TO_SOT_SMD:SOT-23, B.Cu at (129.2, 67.7)
- added R1: 10k, Resistor_SMD:R_0402_1005Metric, B.Cu at (150.2, 59.2)
- added R14: 100k, Resistor_SMD:R_0402_1005Metric, F.Cu at (160.7, 83.0)
- added R22: 5.1k, Resistor_SMD:R_0603_1608Metric, F.Cu at (133.6, 82.8)
- added R26: 0, Resistor_SMD:R_0402_1005Metric, F.Cu at (132.8, 84.2)
- added R28: 200k, Resistor_SMD:R_0603_1608Metric, B.Cu at (162.8, 74.0)
- added R29: 100k, Resistor_SMD:R_0603_1608Metric, B.Cu at (164.3, 74.0)
- added R30: 499k, Resistor_SMD:R_0402_1005Metric, F.Cu at (159.9, 76.0)
- added R35: 0, Resistor_SMD:R_0201_0603Metric, F.Cu at (151.6, 70.7)
- added R44: 0, Resistor_SMD:R_0201_0603Metric, F.Cu at (151.6, 69.3)
- added R51: 0, Resistor_SMD:R_0201_0603Metric, F.Cu at (151.6, 74.2)
- added R52: 0, Resistor_SMD:R_0201_0603Metric, F.Cu at (151.6, 73.5)
- added R53: 0, Resistor_SMD:R_0201_0603Metric, F.Cu at (151.6, 72.8)
- added R54: 0, Resistor_SMD:R_0201_0603Metric, F.Cu at (151.6, 72.1)
- added R55: 0, Resistor_SMD:R_0201_0603Metric, F.Cu at (151.5, 68.6)
- added SW2: B3U-3000P-B, Button_Switch_SMD:SW_SPST_B3U-3000P-B, F.Cu at (168.2, 90.9)
- added SW8: BOOT, Button_Switch_SMD:SW_SPST_CK_KXT3, B.Cu at (156.4, 58.6)
- added U17: TLV62569DDC, Package_TO_SOT_SMD:SOT-23-6, F.Cu at (162.9, 80.2)
- C10, C11: value 22uF -> 100nF; footprint Capacitor_SMD:C_0603_1608Metric -> Capacitor_SMD:C_0402_1005Metric; moved to F.Cu
- C13: value 10uF -> 100nF; footprint Capacitor_SMD:C_0603_1608Metric -> Capacitor_SMD:C_0402_1005Metric; moved to B.Cu
- C14, C16: value 10uF -> 100nF; footprint Capacitor_SMD:C_0603_1608Metric -> Capacitor_SMD:C_0402_1005Metric
- C17: value 22uF -> 1uF; footprint Capacitor_SMD:C_0603_1608Metric -> Capacitor_SMD:C_0402_1005Metric; moved to B.Cu
- C18, C19, C20, C41, C44, C45, C7, C78, C79, C8, D7, D8, R23, U13, U8: moved to F.Cu
- C34: value 1uF -> 10uF; moved to B.Cu
- C4: value 100nF -> 1uF
- C51: footprint Capacitor_SMD:C_0402_1005Metric -> Capacitor_SMD:C_0603_1608Metric
- C55, C57, C58: footprint Capacitor_SMD:C_0402_1005Metric -> Capacitor_SMD:C_0805_2012Metric
- C68, D3, R39, R43, U4: moved to B.Cu
- C82: value 100nF -> 220nF; footprint Capacitor_SMD:C_0402_1005Metric -> Capacitor_SMD:C_0603_1608Metric
- C9: value 22uF -> 1uF; footprint Capacitor_SMD:C_0603_1608Metric -> Capacitor_SMD:C_0402_1005Metric; moved to F.Cu
- J5: footprint Connector_Card:microSD_HC_Hirose_DM3D-SF -> custom-lib:MOLEX_503398-1892
- J6: footprint custom-lib:OK-14GF024-04 -> custom-lib:MOLEX_505550-2420
- L2: value 1uH -> CIGT252010EH1R0MNE
- L3: value 2.2uH -> XFL4020-222ME; footprint Inductor_SMD:L_1206_3216Metric -> Inductor_SMD:L_Coilcraft_XxL4040
- L5: value 2nH -> LQG15HN2N0C02D
- L9: value NRS4018T220MDGJ -> LQM2HPN4R7MG0L; footprint Inductor_SMD:L_Taiyo-Yuden_MD-4040 -> Inductor_SMD:L_1008_2520Metric
- R15: footprint Resistor_SMD:R_0603_1608Metric -> Resistor_SMD:R_0402_1005Metric; moved to B.Cu
- R16, R4: footprint Resistor_SMD:R_0402_1005Metric -> Resistor_SMD:R_0603_1608Metric
- R17: value 5.1k -> 100k; moved to F.Cu
- R19: value 10k -> 100k; moved to F.Cu
- R20, R45, R48, R49, R5: value 10k -> 100k; moved to B.Cu
- R37: value 10k -> 0; footprint Capacitor_SMD:C_0402_1005Metric -> Resistor_SMD:R_0201_0603Metric; moved to F.Cu
- R46, R47: value 10k -> 100k
- R50: value 10k -> 0; footprint Resistor_SMD:R_0402_1005Metric -> Resistor_SMD:R_0201_0603Metric
- R8: value 1M -> 0; footprint Resistor_SMD:R_0402_1005Metric -> Resistor_SMD:R_0201_0603Metric; moved to F.Cu
- SW1: value B3U-3000P -> B3U-3000P-B; footprint Button_Switch_SMD:SW_SPST_B3U-3000P -> Button_Switch_SMD:SW_SPST_B3U-3000P-B
- SW3, SW4: value SW_Push -> B3U-3000P-B; footprint Button_Switch_SMD:SW_SPST_B3U-3000P -> Button_Switch_SMD:SW_SPST_B3U-3000P-B
- U11: value LPS22DF -> ESP32-S3; footprint Package_LGA:ST_HLGA-10_2x2mm_P0.5mm_LayoutBorder3x2y -> Package_DFN_QFN:QFN-56-1EP_7x7mm_P0.4mm_EP4x4mm_ThermalVias
- U3: value TPS62161DSG -> BME280; footprint Package_SON:WSON-8-1EP_2x2mm_P0.5mm_EP0.9x1.6mm_ThermalVias -> Package_LGA:Bosch_LGA-8_2.5x2.5mm_P0.65mm_ClockwisePinNumbering; moved to B.Cu
- moved C29 38.7 mm to (197.1, 70.0), turned to -90 degrees
- moved R12 36.7 mm to (179.0, 102.2), turned to 180 degrees
- moved R11 36.2 mm to (178.0, 101.2)
- moved R9 33.7 mm to (172.6, 104.1), turned to -90 degrees
- moved R37 32.0 mm to (151.6, 70.0), turned to 0 degrees
- moved C11 31.2 mm to (148.4, 67.0), turned to 90 degrees
- moved R45 30.5 mm to (161.5, 95.8), turned to 180 degrees
- moved D4 29.5 mm to (158.2, 76.0), turned to 90 degrees
- moved R13 28.7 mm to (157.3, 76.0), turned to -90 degrees
- moved R5 28.6 mm to (164.9, 94.5)
- moved C10 26.7 mm to (151.4, 75.8), turned to 0 degrees
- moved U15 26.6 mm to (165.7, 94.5), turned to -90 degrees
- moved C52 26.2 mm to (164.7, 92.5)
- moved R20 26.2 mm to (176.6, 65.5), turned to 90 degrees
- moved R15 25.9 mm to (164.9, 102.3), turned to 180 degrees
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Connections:
- C10 pad 1: +BATT -> +1V8
- C11 pad 1: +BATT -> +3V3
- C13 pad 1: +VSW -> +3V3
- C14 pad 1: GND -> Net-(C14-Pad1)
- C14 pad 2: +VSW -> GND
- C16 pad 1: +VSW -> +3V3
- C17 pad 1: +1V8 -> +3V3
- C33 pad 1: GND -> +3V3
- C33 pad 2: +3V3 -> GND
- C34 pad 1: GND -> +3V3
- C34 pad 2: +3V3 -> GND
- C35 pad 1: GND -> Net-(U2-PMID)
- C35 pad 2: +1V8 -> GND
- C4 pad 1: Net-(U2-PMID) -> +3V3
- C41 pad 1: Net-(U7-CHIP_PU) -> Net-(U11-CHIP_PU)
- C9 pad 1: +BATT -> +1V8
- D7 pad 2: /ESP MCU/USB_DP -> /ESP MCU/USB_D+
- D8 pad 2: /ESP MCU/USB_DM -> /ESP MCU/USB_D-
- J2 pad A6: /ESP MCU/USB_DP -> /ESP MCU/USB_D+
- J2 pad A7: /ESP MCU/USB_DM -> /ESP MCU/USB_D-
- J2 pad B6: /ESP MCU/USB_DP -> /ESP MCU/USB_D+
- J2 pad B7: /ESP MCU/USB_DM -> /ESP MCU/USB_D-
- J2 pad S1: unconnected-(J2-SHIELD-PadS1) -> GND
- J6 pad 16: /ESP MCU/IO2 -> /ESP MCU/IO3
- J6 pad 2: /ESP MCU/IO1 -> /ESP MCU/IO2
- J6 pad 21: unconnected-(J6-NC-Pad21) -> (no net)
- L3 pad 1: Net-(U3-SW) -> Net-(U17-SW)
- L5 pad 1: Net-(U7-VDD3P3) -> Net-(C14-Pad1)
- R15 pad 1: +1V8 -> /ESP MCU/EXT_IO11
- R15 pad 2: /USB and Power/1V8_GOOD -> +3V3
- R17 pad 1: Net-(J2-CC2) -> /ESP MCU/EXT_IO12
- R17 pad 2: GND -> +3V3
- R23 pad 2: Net-(U7-CHIP_PU) -> Net-(U11-CHIP_PU)
- R36 pad 1: /ESP MCU/IO5 -> /ESP MCU/IO6
- R37 pad 1: GND -> Net-(U11-GPIO35)
- R37 pad 2: Net-(Q1-G) -> /ESP MCU/MEM_D6
- R46 pad 2: /ESP MCU/IO4 -> /ESP MCU/IO5
- R50 pad 1: GND -> Net-(U11-SPIHD)
- R50 pad 2: /ESP MCU/I2S_SCK -> /ESP MCU/MEM_D3
- R8 pad 1: Net-(U1-FB) -> Net-(U11-GPIO33)
- R8 pad 2: +3V3 -> /ESP MCU/MEM_D4
- SW3 pad 1: /ESP MCU/EXT_IO5 -> GND
- SW3 pad 2: GND -> /ESP MCU/EXT_IO6
- SW4 pad 1: /ESP MCU/EXT_IO6 -> /ESP MCU/EXT_IO7
- U1 pad 12: /USB and Power/1V8_GOOD -> /USB and Power/1V8G
- U1 pad 3: Net-(U1-FB) -> +3V3
- U10 pad 8: /ESP MCU/IO7 -> /ESP MCU/IO8
- U11 pad 1: +3V3 -> /ESP MCU/ESP_ANT
- U11 pad 10: +3V3 -> /ESP MCU/IO2
- U11 pad 2: /IO/ALT_SCL -> Net-(C14-Pad1)
- U11 pad 3: GND -> Net-(C14-Pad1)
- U11 pad 4: /IO/ALT_SDA -> Net-(U11-CHIP_PU)
- U11 pad 5: GND -> /ESP MCU/MCU_SCL
- U11 pad 6: +3V3 -> /ESP MCU/MCU_SDA
- U11 pad 7: /ESP MCU/IO8 -> /ESP MCU/RTC_SCL
- U11 pad 8: GND -> /ESP MCU/RTC_SDA
- U11 pad 9: GND -> /ESP MCU/IO1
- U12 pad 4: /ESP MCU/IO3 -> /ESP MCU/IO4
- U14 pad 13: /ESP MCU/IO4 -> /ESP MCU/IO5
- U16 pad 4: /ESP MCU/IO6 -> /ESP MCU/IO7
- U3 pad 2: +VSW -> +3V3
- U3 pad 3: +VSW -> /IO/TPH_SDA
- U3 pad 4: GND -> /IO/TPH_SCL
- U3 pad 6: +1V8 -> +3V3
- U3 pad 7: Net-(U3-SW) -> GND
- U3 pad 8: /USB and Power/1V8_GOOD -> +3V3
- U8 pad 19: /ESP MCU/I2C0_SDA -> /ESP MCU/I2C0_SCL
- U8 pad 20: /ESP MCU/I2C0_SCL -> /ESP MCU/I2C0_SDA
Routing:
- net /ESP MCU/FSPI_CLK: track 0.00 -> 36.6 mm, vias 0 -> 1
- net /ESP MCU/FSPI_Q: track 0.00 -> 36.3 mm, vias 0 -> 1
- net /ESP MCU/FSPI_D: track 0.00 -> 36.1 mm, vias 0 -> 1
- net /ESP MCU/FSPI_HD: track 0.00 -> 35.9 mm, vias 0 -> 1
- net /ESP MCU/FSPI_CS: track 0.00 -> 35.1 mm, vias 0 -> 1
- net /ESP MCU/FSPI_WP: track 0.00 -> 34.4 mm, vias 0 -> 1
- net /ESP MCU/SD_CLK: track 0.00 -> 30.8 mm, vias 0 -> 1
- net /ESP MCU/SD_D0: track 0.00 -> 30.4 mm, vias 0 -> 1
- net /ESP MCU/SD_D3: track 0.00 -> 29.9 mm, vias 0 -> 1
- net /ESP MCU/SD_D2: track 0.00 -> 29.8 mm, vias 0 -> 1
- net /ESP MCU/SD_D1: track 0.00 -> 29.7 mm, vias 0 -> 1
- net /ESP MCU/SD_CMD: track 0.00 -> 29.6 mm, vias 0 -> 1
- net /ESP MCU/USB_D+: track 0.00 -> 14.2 mm, vias 0 -> 1
- net /ESP MCU/USB_D-: track 0.00 -> 12.7 mm, vias 0 -> 1
- net +3V3: track 0.00 -> 11.0 mm, vias 0 -> 3
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- added copper zone on B.Cu, net GND
- added copper zone on F.Cu, net GND
- added copper zone on In1.Cu, net GND
- added copper zone on In2.Cu, net GND
- added copper zone on In3.Cu, net GND
- added copper zone on In4.Cu, net GND
Other:
- outline, holes or cut-outs redrawn
- board text removed: "BOOT"
- board text removed: "GND"
- board text removed: "RESET"
- board text removed: "TX RX"

Commit message: update
Parts:
- C54, C62, U3: moved to F.Cu
- moved C25 20.2 mm to (153.1, 66.8), turned to 90 degrees
- moved R20 16.8 mm to (159.9, 66.8)
- moved C23 16.5 mm to (158.9, 66.8)
- moved C24 16.5 mm to (158.0, 66.8)
- moved C26 13.7 mm to (156.5, 64.2), turned to 0 degrees
- moved U3 12.2 mm to (160.4, 72.6), turned to 180 degrees
- moved C62 10.3 mm to (162.0, 70.5), turned to 0 degrees
- moved C54 9.44 mm to (159.9, 70.5), turned to 180 degrees
- moved R14 7.46 mm to (155.4, 88.3)
- moved R16 3.29 mm to (135.6, 74.7), turned to 180 degrees
- moved R43 2.40 mm to (144.8, 69.5), turned to 180 degrees
- moved R48 1.01 mm to (162.6, 71.0)
- moved R49 1.01 mm to (163.1, 71.9)
- moved R10 0.97 mm to (160.7, 83.1), turned to 90 degrees
- moved C17 0.90 mm to (139.3, 71.2), turned to -90 degrees
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Connections:
- R46 pad 2: /ESP MCU/IO5 -> /ESP MCU/IO4
- U12 pad 4: /ESP MCU/IO4 -> /ESP MCU/IO5
- U14 pad 13: /ESP MCU/IO5 -> /ESP MCU/IO4
- U16 pad 4: /ESP MCU/IO7 -> /ESP MCU/IO9
Routing:
- net /ESP MCU/I2S_SCK: track 0.00 -> 72.1 mm, vias 0 -> 3
- net /ESP MCU/I2S_WS: track 0.00 -> 65.6 mm, vias 0 -> 3
- net /ESP MCU/I2S_SD: track 0.00 -> 63.4 mm, vias 0 -> 4
- net /ESP MCU/EN: track 0.00 -> 47.6 mm, vias 0 -> 2
- net Net-(U2-QON): track 2.55 -> 24.5 mm, vias 0 -> 2
- net /ESP MCU/IO9: track 0.00 -> 20.9 mm, vias 0 -> 2
- net +3V3: track 11.0 -> 31.0 mm, vias 3 -> 9
- net /ESP MCU/IO1: track 0.00 -> 18.4 mm, vias 1 -> 2
- net GND: track 10.8 -> 28.3 mm, vias 46 -> 53
- net Net-(D2-K): track 0.00 -> 11.8 mm, vias 0 -> 5
- net /ESP MCU/IO8: track 0.00 -> 9.62 mm, vias 0 -> 2
- net Net-(U17-FB): track 0.00 -> 9.13 mm, vias 0 -> 2
- net Net-(D1-A): track 0.00 -> 8.68 mm
- net +VSW: track 2.36 -> 9.95 mm, vias 0 -> 2
- net /ESP MCU/CLK_N: track 0.00 -> 6.00 mm
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
Commit message: old changes
Parts:
- moved R17 0.24 mm to (140.0, 99.1)
Routing:
- net /ESP MCU/IO2: track 3.26 -> 29.3 mm
- net +1V8: track 5.37 -> 25.7 mm, vias 5 -> 6
- net +3V3: track 31.0 -> 48.0 mm, vias 9 -> 12
- net /ESP MCU/EN: track 47.6 -> 46.4 mm
- net /USB and Power/SDA: track 0.59 -> 1.43 mm, vias 1 -> 2
- net Net-(U4-BIN): track 0.00 -> 0.65 mm, vias 0 -> 1
- net Net-(U2-QON): track 24.5 -> 23.9 mm
- net /ESP MCU/EXT_IO12: track 0.00 -> 0.55 mm, vias 0 -> 1
- net +BATT: track 2.85 -> 3.36 mm, vias 1 -> 2
- net /USB and Power/SCL: track 0.81 -> 1.23 mm, vias 1 -> 2
- net Net-(U4-VDD): track 0.00 -> 0.29 mm, vias 0 -> 1
- net GND: vias 53 -> 54
